File: FloraableSchematic/floraable.sch (KiCad schematic (older format))
At the start: 27 parts, among them J1 USB_B, J2 soil moisture sensor, J3 water pump, Q1 IRL1404Z, Q2 IRL1404Z, U1 BA33BC0T, U2 BH1750, U3 NodeMCU, U4 DHT22

Commit message: check for existing devices
Parts:
- removed C3, C5: 100n, Capacitor_SMD:C_0603_1608Metric, symbol Device:C
- removed D2: LED strip, Connector_Molex:Molex_CLIK-Mate_502382-0370_1x03-1MP_P1.25mm_Vertical, symbol Device:LED
- removed R3: 4.7k, Resistor_SMD:R_0603_1608Metric, symbol Device:R
- removed U1: BA33BC0T, Package_TO_SOT_THT:TO-220-3_Vertical, symbol Regulator_Linear:LM7805_TO220
- removed U2: BH1750, BH1750FVI-TR:XDCR_BH1750FVI-TR, symbol Analog_ADC:BH1750
- added C5: 100u, Capacitor_THT:CP_Radial_D5.0mm_P2.00mm, symbol Device:CP
- added J4: LED strip, Connector_PinHeader_2.54mm:PinHeader_1x03_P2.54mm_Horizontal, symbol Connector_Generic:Conn_01x03
- added U1: MCP1702-3302E/TO, Package_TO_SOT_THT:TO-92_Inline, symbol Regulator_Linear:MCP1700-3302E_TO92
- added U2: BH1750_module, floraable:BH1750_module, symbol Analog_ADC:BH1750_module
- C1: footprint Capacitor_SMD:C_0603_1608Metric -> Capacitor_THT:C_Disc_D4.3mm_W1.9mm_P5.00mm
- C2: value 0.33u -> 1u; footprint Capacitor_SMD:C_0603_1608Metric -> Capacitor_THT:C_Disc_D4.3mm_W1.9mm_P5.00mm
- C3: renamed from C4; value 100u -> 1u; footprint Capacitor_SMD:C_0603_1608Metric -> Capacitor_THT:C_Disc_D4.3mm_W1.9mm_P5.00mm
- C4: renamed from C6; footprint Capacitor_SMD:C_0603_1608Metric -> Capacitor_THT:C_Disc_D4.3mm_W1.9mm_P5.00mm
- D1: footprint Diode_SMD:D_SOD-323 -> Diode_THT:D_DO-41_SOD81_P7.62mm_Horizontal
- J2, J3: footprint Connector_Molex:Molex_KK-254_AE-6410-02A_1x02_P2.54mm_Vertical -> Connector_PinHeader_2.54mm:PinHeader_1x02_P2.54mm_Horizontal
- Q1, Q2: footprint Package_TO_SOT_THT:TO-220-3_Horizontal_TabDown -> Package_TO_SOT_THT:TO-220-3_Vertical
- R1, R2: footprint Resistor_SMD:R_0603_1608Metric -> Resistor_THT:R_Axial_DIN0207_L6.3mm_D2.5mm_P10.16mm_Horizontal
- R3: renamed from R4; footprint Resistor_SMD:R_0603_1608Metric -> Resistor_THT:R_Axial_DIN0207_L6.3mm_D2.5mm_P10.16mm_Horizontal
- R4: renamed from R5; footprint Resistor_SMD:R_0603_1608Metric -> Resistor_THT:R_Axial_DIN0207_L6.3mm_D2.5mm_P10.16mm_Horizontal
- R5: renamed from R6; footprint Resistor_SMD:R_0603_1608Metric -> Resistor_THT:R_Axial_DIN0207_L6.3mm_D2.5mm_P10.16mm_Horizontal
- R6: renamed from R7; footprint Resistor_SMD:R_0603_1608Metric -> Resistor_THT:R_Axial_DIN0207_L6.3mm_D2.5mm_P10.16mm_Horizontal
- R7: renamed from R8; footprint Resistor_SMD:R_0603_1608Metric -> Resistor_THT:R_Axial_DIN0207_L6.3mm_D2.5mm_P10.16mm_Horizontal
- R8: renamed from R9; footprint Resistor_SMD:R_0603_1608Metric -> Resistor_THT:R_Axial_DIN0207_L6.3mm_D2.5mm_P10.16mm_Horizontal
- R9: renamed from R10; footprint Resistor_SMD:R_0603_1608Metric -> Resistor_THT:R_Axial_DIN0207_L6.3mm_D2.5mm_P10.16mm_Horizontal
- U3: footprint ESP12E_DEVKIT:ESP12E_DEVKIT -> floraable:newNodeMCU
Connections:
- net +3V3: now also U1.3 (VO), U2.5 (VCC)
- net +5V: now also C5.1, J4.3 (Pin_3), U1.2 (VI)
- net GND: now also U3.GND@0 (GND), U3.GND@2 (GND), U3.GND@3 (GND), C5.2, U1.1 (GND), U2.4 (GND)
- net PUMP: now also R6.1, R7.2
- net SCL: now also U2.3 (SCL)
- net SDA: now also U2.2 (SDA)
- net SOIL: now also J2.1 (Pin_1); no longer J2.2 (Pin_2)
- net TEMPERATURE: now also U3.D8; no longer U3.D3
- net at Q2.2 (D): now also J4.1 (Pin_1)
- net at R1.2: now also J2.2 (Pin_2); no longer J2.1 (Pin_1)
- no-connect marks 0 -> 1
Other:
- moved on the sheet: R3, R4, U3

Commit message: Add files via upload
Connections:
- net TEMPERATURE: now also U3.D5; no longer U3.D8
Other:
- moved on the sheet: C1, C2, C3, C4, C5, D1, J1, J2, J3, J4, Q1, Q2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
